File: mod_synth_mix/schematic/mod_synth_mix.sch (KiCad schematic (older format))
At the start: 24 parts, among them J1 In1, J2 In2, J3 In3, J4 In4, J5 Conn_02x08_Odd_Even, J6 Out, U1 TL072

Commit message: Update mixer
Parts:
- C1, C2: footprint (none) -> Capacitor_THT:CP_Radial_D5.0mm_P2.00mm
- C3, C4: footprint (none) -> Capacitor_THT:C_Disc_D9.0mm_W2.5mm_P5.00mm
- J1, J2, J3, J4, J6: footprint (none) -> Connector_Audio:Jack_3.5mm_QingPu_WQP-PJ398SM_Vertical_CircularHoles
- J5: value Conn_02x08_Odd_Even -> Conn_02x05_Odd_Even; footprint (none) -> Connector_IDC:IDC-Header_2x05_P2.54mm_Vertical; symbol Connector_Generic:Conn_02x08_Odd_Even -> Connector_Generic:Conn_02x05_Odd_Even
- R1, R2, R3, R4, R5, R6, R7, R8: footprint (none) -> Resistor_THT:R_Axial_DIN0207_L6.3mm_D2.5mm_P10.16mm_Horizontal
- RV1, RV2, RV3, RV4, RV5: footprint (none) -> Potentiometer_THT:Potentiometer_Alpha_RD901F-40-00D_Single_Vertical_CircularHoles
- U1: footprint (none) -> Package_DIP:DIP-8_W7.62mm_Socket_LongPads
Changed lines of the file:
@@
 F 0 "J1" H 3057 2775 50  0000 C CNN
 F 1 "In1" H 3057 2684 50  0000 C CNN
-F 2 "" H 3025 2450 50  0001 C CNN
+F 2 "Connector_Audio:Jack_3.5mm_QingPu_WQP-PJ398SM_Vertical_CircularHoles" H 3025 2450 50  0001 C CNN
 F 3 "~" H 3025 2450 50  0001 C CNN
 	1    3025 2450
@@
 F 0 "J2" H 3057 3400 50  0000 C CNN
 F 1 "In2" H 3057 3309 50  0000 C CNN
-F 2 "" H 3025 3075 50  0001 C CNN
+F 2 "Connector_Audio:Jack_3.5mm_QingPu_WQP-PJ398SM_Vertical_CircularHoles" H 3025 3075 50  0001 C CNN
 F 3 "~" H 3025 3075 50  0001 C CNN
 	1    3025 3075
@@
 F 0 "J3" H 3057 3950 50  0000 C CNN
 F 1 "In3" H 3057 3859 50  0000 C CNN
-F 2 "" H 3025 3625 50  0001 C CNN
+F 2 "Connector_Audio:Jack_3.5mm_QingPu_WQP-PJ398SM_Vertical_CircularHoles" H 3025 3625 50  0001 C CNN
 F 3 "~" H 3025 3625 50  0001 C CNN
 	1    3025 3625
@@
 F 0 "J4" H 3057 4625 50  0000 C CNN
 F 1 "In4" H 3057 4534 50  0000 C CNN
-F 2 "" H 3025 4300 50  0001 C CNN
+F 2 "Connector_Audio:Jack_3.5mm_QingPu_WQP-PJ398SM_Vertical_CircularHoles" H 3025 4300 50  0001 C CNN
 F 3 "~" H 3025 4300 50  0001 C CNN
 	1    3025 4300
@@
 F 0 "RV1" V 3768 2450 50  0000 C CNN
 F 1 "100k" V 3859 2450 50  0000 C CNN
-F 2 "" H 3975 2450 50  0001 C CNN
+F 2 "Potentiometer_THT:Potentiometer_Alpha_RD901F-40-00D_Single_Vertical_CircularHoles" H 3975 2450 50  0001 C CNN
 F 3 "~" H 3975 2450 50  0001 C CNN
 	1    3975 2450
@@
 F 0 "RV2" V 3768 3075 50  0000 C CNN
 F 1 "100k" V 3859 3075 50  0000 C CNN
-F 2 "" H 3975 3075 50  0001 C CNN
+F 2 "Potentiometer_THT:Potentiometer_Alpha_RD901F-40-00D_Single_Vertical_CircularHoles" H 3975 3075 50  0001 C CNN
 F 3 "~" H 3975 3075 50  0001 C CNN
 	1    3975 3075
@@
 F 0 "RV3" V 3768 3625 50  0000 C CNN
 F 1 "100k" V 3859 3625 50  0000 C CNN
-F 2 "" H 3975 3625 50  0001 C CNN
+F 2 "Potentiometer_THT:Potentiometer_Alpha_RD901F-40-00D_Single_Vertical_CircularHoles" H 3975 3625 50  0001 C CNN
 F 3 "~" H 3975 3625 50  0001 C CNN
 	1    3975 3625
@@
 F 0 "RV4" V 3768 4300 50  0000 C CNN
 F 1 "100k" V 3859 4300 50  0000 C CNN
-F 2 "" H 3975 4300 50  0001 C CNN
+F 2 "Potentiometer_THT:Potentiometer_Alpha_RD901F-40-00D_Single_Vertical_CircularHoles" H 3975 4300 50  0001 C CNN
 F 3 "~" H 3975 4300 50  0001 C CNN
 	1    3975 4300
@@
 F 0 "R1" V 4718 2600 50  0000 C CNN
 F 1 "47k" V 4809 2600 50  0000 C CNN
-F 2 "" V 4855 2600 50  0001 C CNN
+F 2 "Resistor_THT:R_Axial_DIN0207_L6.3mm_D2.5mm_P10.16mm_Horizontal" V 4855 2600 50  0001 C CNN
 F 3 "~" H 4925 2600 50  0001 C CNN
 	1    4925 2600
@@
 F 0 "R2" V 4718 3225 50  0000 C CNN
 F 1 "47k" V 4809 3225 50  0000 C CNN
-F 2 "" V 4855 3225 50  0001 C CNN
+F 2 "Resistor_THT:R_Axial_DIN0207_L6.3mm_D2.5mm_P10.16mm_Horizontal" V 4855 3225 50  0001 C CNN
 F 3 "~" H 4925 3225 50  0001 C CNN
 	1    4925 3225
@@
 F 0 "R3" V 4718 3775 50  0000 C CNN
 F 1 "47k" V 4809 3775 50  0000 C CNN
-F 2 "" V 4855 3775 50  0001 C CNN
+F 2 "Resistor_THT:R_Axial_DIN0207_L6.3mm_D2.5mm_P10.16mm_Horizontal" V 4855 3775 50  0001 C CNN
 F 3 "~" H 4925 3775 50  0001 C CNN
 	1    4925 3775
@@
 F 0 "R4" V 4718 4450 50  0000 C CNN
 F 1 "47k" V 4809 4450 50  0000 C CNN
-F 2 "" V 4855 4450 50  0001 C CNN
+F 2 "Resistor_THT:R_Axial_DIN0207_L6.3mm_D2.5mm_P10.16mm_Horizontal" V 4855 4450 50  0001 C CNN
 F 3 "~" H 4925 4450 50  0001 C CNN
 	1    4925 4450
@@
 F 0 "J6" H 9295 4375 50  0000 R CNN
 F 1 "Out" H 9295 4284 50  0000 R CNN
-F 2 "" H 9475 4300 50  0001 C CNN
+F 2 "Connector_Audio:Jack_3.5mm_QingPu_WQP-PJ398SM_Vertical_CircularHoles" H 9475 4300 50  0001 C CNN
 F 3 "~" H 9475 4300 50  0001 C CNN
 	1    9475 4300
@@
 F 0 "R5" V 6218 3175 50  0000 C CNN
 F 1 "47k" V 6309 3175 50  0000 C CNN
-F 2 "" V 6355 3175 50  0001 C CNN
+F 2 "Resistor_THT:R_Axial_DIN0207_L6.3mm_D2.5mm_P10.16mm_Horizontal" V 6355 3175 50  0001 C CNN
 F 3 "~" H 6425 3175 50  0001 C CNN
 	1    6425 3175
@@
 F 0 "R7" V 7918 3775 50  0000 C CNN
 F 1 "47k" V 8009 3775 50  0000 C CNN
-F 2 "" V 8055 3775 50  0001 C CNN
+F 2 "Resistor_THT:R_Axial_DIN0207_L6.3mm_D2.5mm_P10.16mm_Horizontal" V 8055 3775 50  0001 C CNN
 F 3 "~" H 8125 3775 50  0001 C CNN
 	1    8125 3775
@@
 F 0 "U1" H 6400 3233 50  0000 C CNN
 F 1 "TL072" H 6400 3324 50  0000 C CNN
-F 2 "" H 6400 3600 50  0001 C CNN
+F 2 "Package_DIP:DIP-8_W7.62mm_Socket_LongPads" H 6400 3600 50  0001 C CNN
 F 3 "http://www.ti.com/lit/ds/symlink/tl071.pdf" H 6400 3600 50  0001 C CNN
 	1    6400 3600
@@
 F 0 "RV5" V 6943 3600 50  0000 C CNN
 F 1 "100k" V 7034 3600 50  0000 C CNN
-F 2 "" H 7150 3600 50  0001 C CNN
+F 2 "Potentiometer_THT:Potentiometer_Alpha_RD901F-40-00D_Single_Vertical_CircularHoles" H 7150 3600 50  0001 C CNN
 F 3 "~" H 7150 3600 50  0001 C CNN
 	1    7150 3600
@@
 F 0 "R6" V 7682 4200 50  0000 C CNN
 F 1 "47k" V 7591 4200 50  0000 C CNN
-F 2 "" V 7405 4200 50  0001 C CNN
+F 2 "Resistor_THT:R_Axial_DIN0207_L6.3mm_D2.5mm_P10.16mm_Horizontal" V 7405 4200 50  0001 C CNN
 F 3 "~" H 7475 4200 50  0001 C CNN
 	1    7475 4200
@@
 F 0 "R8" V 8718 4300 50  0000 C CNN
 F 1 "1k" V 8809 4300 50  0000 C CNN
-F 2 "" V 8855 4300 50  0001 C CNN
+F 2 "Resistor_THT:R_Axial_DIN0207_L6.3mm_D2.5mm_P10.16mm_Horizontal" V 8855 4300 50  0001 C CNN
 F 3 "~" H 8925 4300 50  0001 C CNN
 	1    8925 4300
@@
 	9075 4300 9275 4300
 $Comp
-L Connector_Generic:Conn_02x08_Odd_Even J5
+L Connector_Generic:Conn_02x05_Odd_Even J5
 U 1 1 5D58D29F
-P 4400 5825
-F 0 "J5" H 4450 5200 50  0000 C CNN
-F 1 "Conn_02x08_Odd_Even" H 4450 5291 50  0000 C CNN
-F 2 "" H 4400 5825 50  0001 C CNN
-F 3 "~" H 4400 5825 50  0001 C CNN
-	1    4400 5825
+P 4400 5925
+F 0 "J5" H 4450 5300 50  0000 C CNN
+F 1 "Conn_02x05_Odd_Even" H 4450 5391 50  0000 C CNN
+F 2 "Connector_IDC:IDC-Header_2x05_P2.54mm_Vertical" H 4400 5925 50  0001 C CNN
+F 3 "~" H 4400 5925 50  0001 C CNN
+	1    4400 5925
 	-1   0    0    1
 $EndComp
@@
 F 0 "C1" H 5093 5571 50  0000 L CNN
 F 1 "10uf" H 5093 5480 50  0000 L CNN
-F 2 "" H 5013 5375 50  0001 C CNN
+F 2 "Capacitor_THT:CP_Radial_D5.0mm_P2.00mm" H 5013 5375 50  0001 C CNN
 F 3 "~" H 4975 5525 50  0001 C CNN
 	1    4975 5525
@@
 F 0 "C3" H 5465 5571 50  0000 L CNN
 F 1 "100nf" H 5465 5480 50  0000 L CNN
-F 2 "" H 5388 5375 50  0001 C CNN
+F 2 "Capacitor_THT:C_Disc_D9.0mm_W2.5mm_P5.00mm" H 5388 5375 50  0001 C CNN
 F 3 "~" H 5350 5525 50  0001 C CNN
 	1    5350 5525
@@
 F 0 "C2" H 5093 6271 50  0000 L CNN
 F 1 "10uf" H 5093 6180 50  0000 L CNN
-F 2 "" H 5013 6075 50  0001 C CNN
+F 2 "Capacitor_THT:CP_Radial_D5.0mm_P2.00mm" H 5013 6075 50  0001 C CNN
 F 3 "~" H 4975 6225 50  0001 C CNN
 	1    4975 6225
@@
 F 0 "C4" H 5465 6271 50  0000 L CNN
 F 1 "100nf" H 5465 6180 50  0000 L CNN
-F 2 "" H 5388 6075 50  0001 C CNN
+F 2 "Capacitor_THT:C_Disc_D9.0mm_W2.5mm_P5.00mm" H 5388 6075 50  0001 C CNN
 F 3 "~" H 5350 6225 50  0001 C CNN
 	1    5350 6225
