File: mod_synth_div/schematic/mod_synth_div.kicad_pcb (KiCad board)
At the start: 2 copper layers, 50.8 x 109.2 mm, 68 parts, among them J1 In, J10 Conn_01x05_Female, J11 Conn_01x05_Male, J12 Conn_01x05_Female, J13 Conn_01x05_Male, J2 Rst, J3 Conn_02x08_Odd_Even, J4 1/2, J5 1/4, J6 1/8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

Commit message: Add PCB connectors
Parts:
- C3, C5, J3: moved to B.Cu
- moved J3 2.54 mm to (69.8, 169.5), turned to 0 degrees
Connections:
- D4 pad 1: GND -> /GND_PCB_B
- D5 pad 1: GND -> /GND_PCB_B
- D6 pad 1: GND -> /GND_PCB_B
- D7 pad 1: GND -> /GND_PCB_B
- D8 pad 1: GND -> /GND_PCB_B
- D9 pad 1: GND -> /GND_PCB_B
- J1 pad S: GND -> /GND_PCB_B
- J10 pad 1: Net-(J10-Pad1) -> /2_PCB_A
- J10 pad 2: Net-(J10-Pad2) -> /3_PCB_A
- J10 pad 3: Net-(J10-Pad3) -> +5V
- J10 pad 4: Net-(J10-Pad4) -> GND
- J10 pad 5: Net-(J10-Pad5) -> /4_PCB_A
- J11 pad 1: Net-(J11-Pad1) -> /2_PCB_B
- J11 pad 2: Net-(J11-Pad2) -> /3_PCB_B
- J11 pad 3: Net-(J11-Pad3) -> /5V_PCB_B
- J11 pad 4: Net-(J11-Pad4) -> /GND_PCB_B
- J11 pad 5: Net-(J11-Pad5) -> /4_PCB_B
- J12 pad 1: Net-(J12-Pad1) -> /IN_PCB_A
- J12 pad 2: Net-(J12-Pad2) -> /RST_PCB_A
- J12 pad 3: Net-(J12-Pad3) -> /OUT_PCB_A
- J12 pad 4: Net-(J12-Pad4) -> /0_PCB_A
- J12 pad 5: Net-(J12-Pad5) -> /1_PCB_A
- J13 pad 1: Net-(J13-Pad1) -> /IN_PCB_B
- J13 pad 2: Net-(J13-Pad2) -> /RST_PCB_B
- J13 pad 3: Net-(J13-Pad3) -> /OUT_PCB_B
- J13 pad 4: Net-(J13-Pad4) -> /0_PCB_B
- J13 pad 5: Net-(J13-Pad5) -> /1_PCB_B
- J2 pad S: GND -> /GND_PCB_B
- J4 pad S: GND -> /GND_PCB_B
- J5 pad S: GND -> /GND_PCB_B
- J6 pad S: GND -> /GND_PCB_B
- J7 pad S: GND -> /GND_PCB_B
- J8 pad S: GND -> /GND_PCB_B
- J9 pad S: GND -> /GND_PCB_B
- Q10 pad 1: +5V -> /5V_PCB_B
- Q11 pad 1: +5V -> /5V_PCB_B
- Q2 pad 2: Net-(Q2-Pad2) -> /RST_PCB_A
- Q3 pad 2: Net-(Q3-Pad2) -> /IN_PCB_A
- Q5 pad 1: Net-(Q5-Pad1) -> /OUT_PCB_A
- Q6 pad 1: +5V -> /5V_PCB_B
- Q7 pad 1: +5V -> /5V_PCB_B
- Q8 pad 1: +5V -> /5V_PCB_B
- Q9 pad 1: +5V -> /5V_PCB_B
- R11 pad 1: Net-(Q5-Pad1) -> /OUT_PCB_A
- R12 pad 1: Net-(R12-Pad1) -> /0_PCB_B
- R13 pad 1: Net-(R13-Pad1) -> /1_PCB_B
- R14 pad 1: Net-(R14-Pad1) -> /2_PCB_B
- R15 pad 1: Net-(R15-Pad1) -> /3_PCB_B
- R16 pad 1: Net-(R16-Pad1) -> /4_PCB_B
- R17 pad 1: Net-(Q5-Pad1) -> /OUT_PCB_B
- R3 pad 2: Net-(Q2-Pad2) -> /RST_PCB_B
- R4 pad 1: Net-(Q3-Pad2) -> /IN_PCB_B
- R9 pad 2: Net-(Q2-Pad2) -> /RST_PCB_A
- U1 pad 11: Net-(R13-Pad1) -> /1_PCB_A
- U1 pad 12: Net-(R12-Pad1) -> /0_PCB_A
- U1 pad 5: Net-(R16-Pad1) -> /4_PCB_A
- U1 pad 6: Net-(R15-Pad1) -> /3_PCB_A
- U1 pad 9: Net-(R14-Pad1) -> /2_PCB_A
Routing:
- net /RST_PCB_B: track 0.00 -> 38.7 mm
- net /2_PCB_B: track 0.00 -> 32.1 mm
- net /OUT_PCB_B: track 0.00 -> 30.5 mm
- net /IN_PCB_B: track 0.00 -> 29.7 mm
- net /5V_PCB_B: track 0.00 -> 22.3 mm
- net /1_PCB_B: track 0.00 -> 20.7 mm
- net /3_PCB_B: track 0.00 -> 19.3 mm
- net /4_PCB_B: track 0.00 -> 19.2 mm
- net /0_PCB_B: track 0.00 -> 19.1 mm
- net Net-(Q9-Pad3): track 0.00 -> 16.6 mm
- net Net-(Q8-Pad3): track 0.00 -> 16.6 mm
- net Net-(Q7-Pad3): track 0.00 -> 16.6 mm
- net Net-(Q6-Pad3): track 0.00 -> 16.2 mm
- net Net-(Q11-Pad3): track 0.00 -> 15.9 mm
- net Net-(Q10-Pad3): track 0.00 -> 15.5 mm
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- added copper zone on B.Cu, net /GND_PCB_B
- added copper zone on F.Cu, net /GND_PCB_B
- added copper zone on B.Cu, net GND

Commit message: Layout tracks for divider
Parts:
- C1, C2, C3, C4, C5, D3, J3, Q1, Q2, Q3, Q4, Q5, R1, R10, R11, R2, R5, R6, R7, R8, R9, U1: moved to F.Cu
- moved J3 17.8 mm to (69.8, 151.8)
- moved R8 14.7 mm to (60.5, 85.1), turned to 90 degrees
- moved R6 10.9 mm to (64.3, 85.1), turned to 90 degrees
- moved R11 10.7 mm to (67.6, 74.9), turned to 270 degrees
- moved R5 10.4 mm to (60.5, 93.2), turned to 270 degrees
- moved R1 10.3 mm to (74.9, 93.3), turned to 270 degrees
- moved R7 10.2 mm to (74.7, 85.1), turned to 90 degrees
- moved R2 10.2 mm to (71.1, 93.3), turned to 270 degrees
- moved R9 10.0 mm to (64.3, 103.4), turned to 90 degrees
- moved D3 7.75 mm to (67.6, 95.8), turned to 270 degrees
- moved U1 7.62 mm to (66.7, 118.1), turned to 0 degrees
- moved R10 3.56 mm to (71.1, 85.1)
- moved Q5 0.80 mm to (72.1, 89.7)
- moved Q4 0.77 mm to (60.5, 89.7)
- moved Q1 0.76 mm to (66.3, 89.7)
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Routing:
- net +12V: track 0.00 -> 168.9 mm
- net /5V_PCB_B: track 22.3 -> 103.6 mm
- net +5V: track 0.00 -> 69.2 mm
- net /2_PCB_A: track 0.00 -> 61.5 mm
- net Net-(Q3-Pad1): track 0.00 -> 53.7 mm
- net /4_PCB_A: track 0.00 -> 46.8 mm
- net /OUT_PCB_A: track 0.00 -> 45.3 mm
- net /RST_PCB_A: track 0.00 -> 42.9 mm
- net /IN_PCB_A: track 0.00 -> 42.9 mm
- net Net-(D3-Pad2): track 0.00 -> 41.0 mm
- net Net-(Q4-Pad1): track 0.00 -> 40.8 mm
- net /3_PCB_A: track 0.00 -> 36.9 mm
- net Net-(C1-Pad1): track 0.00 -> 21.5 mm
- net Net-(Q2-Pad1): track 0.00 -> 21.4 mm
- net /1_PCB_A: track 0.00 -> 20.2 mm
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
Commit message: Rotate connector
Parts:
- moved J3 17.8 mm to (72.4, 169.4), turned to 180 degrees
Routing:
- net +12V: track 168.9 -> 180.9 mm
- net +5V: track 69.2 -> 71.0 mm
- net GND: vias 2 -> 3
Changed lines of the file:
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@@
     (thickness 1.6)
     (drawings 9)
-    (tracks 357)
+    (tracks 363)
     (zones 0)
     (modules 68)
@@
     (solder_mask_min_width 0.25)
     (aux_axis_origin 0 0)
-    (visible_elements FFFFFF7F)
+    (visible_elements 7FFFFFFF)
     (pcbplotparams
       (layerselection 0x010fc_ffffffff)
@@
   )
   (module Connector_IDC:IDC-Header_2x08_P2.54mm_Vertical (layer F.Cu)
-    (at 69.85 151.765)
+    (at 72.39 169.418 180)
     (descr "Through hole straight IDC box header, 2x08, 2.54mm pitch, double rows")
     (tags "Through hole IDC box header THT 2x08 2.54mm double row")
@@
       (effects (font (size 1 1) (thickness 0.15)))
     )
-    (pad 16 thru_hole oval (at 2.54 17.78) (size 1.7272 1.7272) (drill 1.016) (layers *.Cu *.Mask)
+    (pad 16 thru_hole oval (at 2.54 17.78 180) (size 1.7272 1.7272) (drill 1.016) (layers *.Cu *.Mask)
       (net 17 "Net-(J3-Pad16)"))
-    (pad 15 thru_hole oval (at 0 17.78) (size 1.7272 1.7272) (drill 1.016) (layers *.Cu *.Mask)
+    (pad 15 thru_hole oval (at 0 17.78 180) (size 1.7272 1.7272) (drill 1.016) (layers *.Cu *.Mask)
       (net 18 "Net-(J3-Pad15)"))
-    (pad 14 thru_hole oval (at 2.54 15.24) (size 1.7272 1.7272) (drill 1.016) (layers *.Cu *.Mask)
+    (pad 14 thru_hole oval (at 2.54 15.24 180) (size 1.7272 1.7272) (drill 1.016) (layers *.Cu *.Mask)
       (net 19 "Net-(J3-Pad14)"))
-    (pad 13 thru_hole oval (at 0 15.24) (size 1.7272 1.7272) (drill 1.016) (layers *.Cu *.Mask)
+    (pad 13 thru_hole oval (at 0 15.24 180) (size 1.7272 1.7272) (drill 1.016) (layers *.Cu *.Mask)
       (net 20 "Net-(J3-Pad13)"))
-    (pad 12 thru_hole oval (at 2.54 12.7) (size 1.7272 1.7272) (drill 1.016) (layers *.Cu *.Mask)
+    (pad 12 thru_hole oval (at 2.54 12.7 180) (size 1.7272 1.7272) (drill 1.016) (layers *.Cu *.Mask)
       (net 4 +5V))
-    (pad 11 thru_hole oval (at 0 12.7) (size 1.7272 1.7272) (drill 1.016) (layers *.Cu *.Mask)
+    (pad 11 thru_hole oval (at 0 12.7 180) (size 1.7272 1.7272) (drill 1.016) (layers *.Cu *.Mask)
       (net 4 +5V))
-    (pad 10 thru_hole oval (at 2.54 10.16) (size 1.7272 1.7272) (drill 1.016) (layers *.Cu *.Mask)
+    (pad 10 thru_hole oval (at 2.54 10.16 180) (size 1.7272 1.7272) (drill 1.016) (layers *.Cu *.Mask)
       (net 3 +12V))
-    (pad 9 thru_hole oval (at 0 10.16) (size 1.7272 1.7272) (drill 1.016) (layers *.Cu *.Mask)
+    (pad 9 thru_hole oval (at 0 10.16 180) (size 1.7272 1.7272) (drill 1.016) (layers *.Cu *.Mask)
       (net 3 +12V))
-    (pad 8 thru_hole oval (at 2.54 7.62) (size 1.7272 1.7272) (drill 1.016) (layers *.Cu *.Mask)
+    (pad 8 thru_hole oval (at 2.54 7.62 180) (size 1.7272 1.7272) (drill 1.016) (layers *.Cu *.Mask)
       (net 1 GND))
-    (pad 7 thru_hole oval (at 0 7.62) (size 1.7272 1.7272) (drill 1.016) (layers *.Cu *.Mask)
+    (pad 7 thru_hole oval (at 0 7.62 180) (size 1.7272 1.7272) (drill 1.016) (layers *.Cu *.Mask)
       (net 1 GND))
-    (pad 6 thru_hole oval (at 2.54 5.08) (size 1.7272 1.7272) (drill 1.016) (layers *.Cu *.Mask)
+    (pad 6 thru_hole oval (at 2.54 5.08 180) (size 1.7272 1.7272) (drill 1.016) (layers *.Cu *.Mask)
       (net 1 GND))
-    (pad 5 thru_hole oval (at 0 5.08) (size 1.7272 1.7272) (drill 1.016) (layers *.Cu *.Mask)
+    (pad 5 thru_hole oval (at 0 5.08 180) (size 1.7272 1.7272) (drill 1.016) (layers *.Cu *.Mask)
       (net 1 GND))
-    (pad 4 thru_hole oval (at 2.54 2.54) (size 1.7272 1.7272) (drill 1.016) (layers *.Cu *.Mask)
+    (pad 4 thru_hole oval (at 2.54 2.54 180) (size 1.7272 1.7272) (drill 1.016) (layers *.Cu *.Mask)
       (net 1 GND))
-    (pad 3 thru_hole oval (at 0 2.54) (size 1.7272 1.7272) (drill 1.016) (layers *.Cu *.Mask)
+    (pad 3 thru_hole oval (at 0 2.54 180) (size 1.7272 1.7272) (drill 1.016) (layers *.Cu *.Mask)
       (net 1 GND))
-    (pad 2 thru_hole oval (at 2.54 0) (size 1.7272 1.7272) (drill 1.016) (layers *.Cu *.Mask)
+    (pad 2 thru_hole oval (at 2.54 0 180) (size 1.7272 1.7272) (drill 1.016) (layers *.Cu *.Mask)
       (net 21 "Net-(J3-Pad2)"))
-    (pad 1 thru_hole rect (at 0 0) (size 1.7272 1.7272) (drill 1.016) (layers *.Cu *.Mask)
+    (pad 1 thru_hole rect (at 0 0 180) (size 1.7272 1.7272) (drill 1.016) (layers *.Cu *.Mask)
       (net 22 "Net-(J3-Pad1)"))
     (model ${KISYS3DMOD}/Connector_IDC.3dshapes/IDC-Header_2x08_P2.54mm_Vertical.wrl
@@
   (segment (start 73.152 91.948) (end 73.152 94.051006) (width 0.25) (layer F.Cu) (net 1))
   (via (at 72.603516 94.59949) (size 0.8) (drill 0.4) (layers F.Cu B.Cu) (net 1))
+  (via (at 65.532 149.098) (size 0.8) (drill 0.4) (layers F.Cu B.Cu) (net 1))
   (segment (start 71.12 101.839998) (end 71.12 94.47637) (width 0.25) (layer F.Cu) (net 2))
   (segment (start 66.675 106.284998) (end 71.12 101.839998) (width 0.25) (layer F.Cu) (net 2))
@@
   (segment (start 66.675 109.22) (end 66.675 106.284998) (width 0.25) (layer F.Cu) (net 2))
   (segment (start 71.12 93.345) (end 74.93 93.345) (width 0.25) (layer B.Cu) (net 2))
-  (segment (start 71.071314 161.925) (end 72.39 161.925) (width 0.25) (layer F.Cu) (net 3))
-  (segment (start 69.85 161.925) (end 71.071314 161.925) (width 0.25) (layer F.Cu) (net 3))
-  (segment (start 60.96 155.355) (end 60.96 154.305) (width 0.25) (layer F.Cu) (net 3))
-  (segment (start 66.666401 161.061401) (end 60.96 155.355) (width 0.25) (layer F.Cu) (net 3))
-  (segment (start 68.986401 161.061401) (end 66.666401 161.061401) (width 0.25) (layer F.Cu) (net 3))
-  (segment (start 69.85 161.925) (end 68.986401 161.061401) (width 0.25) (layer F.Cu) (net 3))
   (segment (start 60.96 151.765) (end 73.025 139.7) (width 0.25) (layer F.Cu) (net 3))
   (segment (start 60.96 154.305) (end 60.96 151.765) (width 0.25) (layer F.Cu) (net 3))
@@
   (segment (start 74.93 102.37363) (end 76.055001 101.248629) (width 0.25) (layer B.Cu) (net 3))
   (segment (start 74.93 103.505) (end 74.93 102.37363) (width 0.25) (layer B.Cu) (net 3))
-  (segment (start 71.168686 164.465) (end 69.85 164.465) (width 0.25) (layer F.Cu) (net 4))
-  (segment (start 72.39 164.465) (end 71.168686 164.465) (width 0.25) (layer F.Cu) (net 4))
-  (segment (start 69.85 164.465) (end 62.865 164.465) (width 0.25) (layer F.Cu) (net 4))
+  (segment (start 69.85 159.258) (end 72.39 159.258) (width 0.25) (layer F.Cu) (net 3))
+  (segment (start 73.253599 158.394401) (end 72.39 159.258) (width 0.25) (layer F.Cu) (net 3))
+  (segment (start 73.578601 151.067471) (end 73.578601 158.069399) (width 0.25) (layer F.Cu) (net 3))
+  (segment (start 72.960529 150.449399) (end 73.578601 151.067471) (width 0.25) (layer F.Cu) (net 3))
+  (segment (start 69.279471 150.449399) (end 72.960529 150.449399) (width 0.25) (layer F.Cu) (net 3))
+  (segment (start 73.578601 158.069399) (end 73.253599 158.394401) (width 0.25) (layer F.Cu) (net 3))
+  (segment (start 61.035001 155.430001) (end 64.298869 155.430001) (width 0.25) (layer F.Cu) (net 3))
+  (segment (start 64.298869 155.430001) (end 69.279471 150.449399) (width 0.25) (layer F.Cu) (net 3))
+  (segment (start 60.96 155.355) (end 61.035001 155.430001) (width 0.25) (layer F.Cu) (net 3))
+  (segment (start 60.96 154.305) (end 60.96 155.355) (width 0.25) (layer F.Cu) (net 3))
   (segment (start 59.834999 157.879997) (end 62.738 160.782998) (width 0.25) (layer F.Cu) (net 4))
   (segment (start 59.834999 149.495001) (end 59.834999 157.879997) (width 0.25) (layer F.Cu) (net 4))
@@
   (segment (start 60.96 145.099998) (end 72.225001 133.834997) (width 0.25) (layer F.Cu) (net 4))
   (segment (start 60.96 147.32) (end 60.96 145.099998) (width 0.25) (layer F.Cu) (net 4))
+  (segment (start 65.785002 160.782998) (end 69.85 156.718) (width 0.25) (layer F.Cu) (net 4))
+  (segment (start 62.738 160.782998) (end 65.785002 160.782998) (width 0.25) (layer F.Cu) (net 4))
+  (segment (start 69.85 156.718) (end 72.39 156.718) (width 0.25) (layer F.Cu) (net 4))
   (segment (start 46.355 80.615) (end 53.945 73.025) (width 0.25) (layer F.Cu) (net 5))
   (segment (start 46.355 82.55) (end 46.355 80.615) (width 0.25) (layer F.Cu) (net 5))
@@
   (segment (start 40.099999 97.299999) (end 43.324999 97.299999) (width 0.25) (layer F.Cu) (net 59))
   (segment (start 27.94 113.665) (end 36.974999 104.630001) (width 0.25) (layer F.Cu) (net 59))
-  (segment (start 59.86 161.29) (end 60.96 161.29) (width 0.25) (layer F.Cu) (net 60))
-  (segment (start 59.784999 161.365001) (end 59.86 161.29) (width 0.25) (layer F.Cu) (net 60))
-  (segment (start 59.784999 172.014001) (end 59.784999 161.365001) (width 0.25) (layer F.Cu) (net 60))
-  (segment (start 60.395999 172.625001) (end 59.784999 172.014001) (width 0.25) (layer F.Cu) (net 60))
-  (segment (start 71.069129 172.625001) (end 60.395999 172.625001) (width 0.25) (layer F.Cu) (net 60))
-  (segment (start 74.295 169.39913) (end 71.069129 172.625001) (width 0.25) (layer F.Cu) (net 60))
-  (segment (start 74.295 135.89) (end 74.295 169.39913) (width 0.25) (layer F.Cu) (net 60))
+  (segment (start 74.295 169.39913) (end 74.295 135.89) (width 0.25) (layer F.Cu) (net 60))
+  (segment (start 60.96 161.29) (end 59.86 161.29) (width 0.25) (layer F.Cu) (net 60))
+  (segment (start 59.86 161.29) (end 59.784999 161.365001) (width 0.25) (layer F.Cu) (net 60))
+  (segment (start 74.295 169.825202) (end 74.295 169.39913) (width 0.25) (layer F.Cu) (net 60))
+  (segment (start 59.784999 161.365001) (end 59.784999 172.014001) (width 0.25) (layer F.Cu) (net 60))
+  (segment (start 59.784999 172.014001) (end 60.395999 172.625001) (width 0.25) (layer F.Cu) (net 60))
+  (segment (start 60.395999 172.625001) (end 71.495201 172.625001) (width 0.25) (layer F.Cu) (net 60))
+  (segment (start 71.495201 172.625001) (end 74.295 169.825202) (width 0.25) (layer F.Cu) (net 60))
   (segment (start 43.650001 143.345001) (end 44.45 144.145) (width 0.25) (layer F.Cu) (net 61))
   (segment (start 43.324999 143.019999) (end 43.650001 143.345001) (width 0.25) (layer F.Cu) (net 61))
