File: mod_synth_lfo_full/schematic/mod_synth_lfo_full.sch (KiCad schematic (older format))
At the start: 75 parts, among them J1 CV, J2 Conn_02x08_Odd_Even, J3 SIN, J4 COS, J5 TRI, J6 SQR, J7 RAMP UP, J8 RAMP DOWN, Q1 BC550, Q2 BC550, Q3 BC550, Q4 BC550, Q5 BC550, U1 TL072, U2 TL072, U3 TL072, U4 TL074

Commit message: Convert SMT LFO to multi-PCB
Parts:
- R1, R10, R11, R12, R13, R14, R15, R16, R17, R19, R2, R20, R21, R22, R23, R24, R25, R26, R27, R28, R29, R3, R30, R32, R33, R34, R35, R36, R37, R38, R39, R4, R40, R41, R42, R5, R6, R7, R8, R9: footprint Resistor_SMD:R_1206_3216Metric_Pad1.42x1.75mm_HandSolder -> Resistor_THT:R_Axial_DIN0207_L6.3mm_D2.5mm_P10.16mm_Horizontal
- U1, U2, U3: footprint st_package_so:SOIC-8 -> Package_DIP:DIP-8_W7.62mm_Socket_LongPads
- U4: footprint st_package_so:SOIC-14 -> Package_DIP:DIP-14_W7.62mm_Socket_LongPads
