File: mod_synth_out_nophones/schematic/mod_synth_out_nophones.sch (KiCad schematic (older format))
At the start: 50 parts, among them J1 L IN, J2 R IN, J3 Conn_02x08_Odd_Even, J5 L OUT, J6 R OUT, J7 Conn_01x07_Female, J8 Conn_01x07_Male, Q1 2N3904, Q2 2N3904, U1 TL072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

Commit message: Layout components
Parts:
- J7: value Conn_01x07_Female -> Conn_01x11_Female; footprint Connector_PinSocket_2.54mm:PinSocket_1x07_P2.54mm_Vertical -> Connector_PinSocket_2.54mm:PinSocket_1x11_P2.54mm_Vertical; symbol Connector:Conn_01x07_Female -> Connector:Conn_01x11_Female
- J8: value Conn_01x07_Male -> Conn_01x011_Male; footprint Connector_PinHeader_2.54mm:PinHeader_1x07_P2.54mm_Vertical -> Connector_PinHeader_2.54mm:PinHeader_1x11_P2.54mm_Vertical; symbol Connector:Conn_01x07_Male -> Connector:Conn_01x11_Male
Connections:
- net +12V: now also C10.2, U1.8 (V+)
- net +12_PCB_B: no longer C10.2, U1.8 (V+)
- net -12V: now also C7.1, U1.4 (V-)
- net -12_PCB_B: no longer C7.1, U1.4 (V-)
- net GND: now also C10.1, C7.2
- net GND_PCB_B: no longer C10.1, C7.2
- net B_IN_L: now reaches C5.2, R3.2, U1.2 (-)
- net B_IN_L: now also J7.4 (Pin_4); no longer R1.1
- net B_IN_R: now reaches C6.2, R4.2, U1.6 (-)
- net B_IN_R: now also J7.5 (Pin_5); no longer R2.1
- net A_RAW_ML: now reaches RV1.3
- net A_RAW_ML: now also J8.8 (Pin_8); no longer C8.2
- net A_RAW_MR: now reaches RV1.6
- net A_RAW_MR: now also J8.9 (Pin_9); no longer C9.2
- net A_IN_L: now reaches J8.4 (Pin_4)
- net A_IN_L: now also R1.1
- net A_IN_R: now reaches J8.5 (Pin_5)
- net A_IN_R: now also R2.1
- new net B_RAW_ML: C8.2, J7.8 (Pin_8)
- new net B_RAW_MR: C9.2, J7.9 (Pin_9)
Other:
- moved on the sheet: C10, C5, C6, C7, C8, C9, R3, R4, RV1A, RV1B, U1A, U1B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
