File: mod_synth_sw/schematic/mod_synth_sw.kicad_pcb (KiCad board)
At the start: 2 copper layers, 62.2 x 109.2 mm, 52 parts, among them J1 Conn_02x08_Odd_Even, J10 Conn_01x06_Male, J11 Conn_01x07_Female, J12 Conn_01x07_Male, J2 CLK, J3 RST, J4 I/O, J5 I/O 1, J6 I/O 2, J7 I/O 3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

Commit message: Update values
Parts:
- C1: value C -> 100n
- R1, R2, R8, R9: value R -> 47k
- R10: value R -> 2k7
- R11, R12, R13, R14, R15: value R -> 1k
- R3, R4, R5, R6, R7: value R -> 10k
Changed lines of the file:
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@@
       (effects (font (size 1 1) (thickness 0.15)) (justify mirror))
     )
-    (fp_text value R (at 5.08 -2.37 90) (layer B.Fab)
+    (fp_text value 1k (at 5.08 -2.37 90) (layer B.Fab)
       (effects (font (size 1 1) (thickness 0.15)) (justify mirror))
     )
@@
       (effects (font (size 1 1) (thickness 0.15)) (justify mirror))
     )
-    (fp_text value R (at 5.08 -2.37 270) (layer B.Fab)
+    (fp_text value 1k (at 5.08 -2.37 270) (layer B.Fab)
       (effects (font (size 1 1) (thickness 0.15)) (justify mirror))
     )
@@
       (effects (font (size 1 1) (thickness 0.15)) (justify mirror))
     )
-    (fp_text value R (at 5.08 -2.37 90) (layer B.Fab)
+    (fp_text value 1k (at 5.08 -2.37 90) (layer B.Fab)
       (effects (font (size 1 1) (thickness 0.15)) (justify mirror))
     )
@@
       (effects (font (size 1 1) (thickness 0.15)) (justify mirror))
     )
-    (fp_text value R (at 5.08 -2.37 90) (layer B.Fab)
+    (fp_text value 1k (at 5.08 -2.37 90) (layer B.Fab)
       (effects (font (size 1 1) (thickness 0.15)) (justify mirror))
     )
@@
       (effects (font (size 1 1) (thickness 0.15)) (justify mirror))
     )
-    (fp_text value R (at 5.08 -2.37 270) (layer B.Fab)
+    (fp_text value 1k (at 5.08 -2.37 270) (layer B.Fab)
       (effects (font (size 1 1) (thickness 0.15)) (justify mirror))
     )
@@
       (effects (font (size 1 1) (thickness 0.15)) (justify mirror))
     )
-    (fp_text value R (at 5.08 -2.37 270) (layer B.Fab)
+    (fp_text value 2k7 (at 5.08 -2.37 270) (layer B.Fab)
       (effects (font (size 1 1) (thickness 0.15)) (justify mirror))
     )
@@
       (effects (font (size 1 1) (thickness 0.15)))
     )
-    (fp_text value R (at 5.08 2.37 270) (layer F.Fab)
+    (fp_text value 47k (at 5.08 2.37 270) (layer F.Fab)
       (effects (font (size 1 1) (thickness 0.15)))
     )
@@
       (effects (font (size 1 1) (thickness 0.15)))
     )
-    (fp_text value R (at 5.08 2.37 90) (layer F.Fab)
+    (fp_text value 47k (at 5.08 2.37 90) (layer F.Fab)
       (effects (font (size 1 1) (thickness 0.15)))
     )
@@
       (effects (font (size 1 1) (thickness 0.15)))
     )
-    (fp_text value R (at 5.08 2.37 90) (layer F.Fab)
+    (fp_text value 10k (at 5.08 2.37 90) (layer F.Fab)
       (effects (font (size 1 1) (thickness 0.15)))
     )
@@
       (effects (font (size 1 1) (thickness 0.15)))
     )
-    (fp_text value R (at 5.08 2.37 90) (layer F.Fab)
+    (fp_text value 10k (at 5.08 2.37 90) (layer F.Fab)
       (effects (font (size 1 1) (thickness 0.15)))
     )
@@
       (effects (font (size 1 1) (thickness 0.15)))
     )
-    (fp_text value R (at 5.08 2.37 90) (layer F.Fab)
+    (fp_text value 10k (at 5.08 2.37 90) (layer F.Fab)
       (effects (font (size 1 1) (thickness 0.15)))
     )
@@
       (effects (font (size 1 1) (thickness 0.15)))
     )
-    (fp_text value R (at 5.08 2.37 90) (layer F.Fab)
+    (fp_text value 10k (at 5.08 2.37 90) (layer F.Fab)
       (effects (font (size 1 1) (thickness 0.15)))
     )
@@
       (effects (font (size 1 1) (thickness 0.15)))
     )
-    (fp_text value R (at 5.08 2.37 270) (layer F.Fab)
+    (fp_text value 10k (at 5.08 2.37 270) (layer F.Fab)
       (effects (font (size 1 1) (thickness 0.15)))
     )
@@
       (effects (font (size 1 1) (thickness 0.15)) (justify mirror))
     )
-    (fp_text value R (at 5.08 -2.37 270) (layer B.Fab)
+    (fp_text value 47k (at 5.08 -2.37 270) (layer B.Fab)
       (effects (font (size 1 1) (thickness 0.15)) (justify mirror))
     )
@@
       (effects (font (size 1 1) (thickness 0.15)) (justify mirror))
     )
-    (fp_text value R (at 5.08 -2.37 270) (layer B.Fab)
+    (fp_text value 47k (at 5.08 -2.37 270) (layer B.Fab)
       (effects (font (size 1 1) (thickness 0.15)) (justify mirror))
     )
@@
       (effects (font (size 1 1) (thickness 0.15)))
     )
-    (fp_text value C (at 2.5 2.5) (layer F.Fab)
-      (effects (font (size 1 1) (thickness 0.15)))
-    )
+    (fp_text value 100n (at 2.5 2.5) (layer F.Fab)
+      (effects (font (size 1 1) (thickness 0.15)))
+    )
