File: mod_synth_kick/schematic/mod_synth_kick.kicad_pcb (KiCad board)
At the start: 2 copper layers, 41.9 x 109.2 mm, 39 parts, among them J1 Trigger, J2 Out, J3 Conn_02x08_Odd_Even, J4 Conn_01x05_Female, J5 Conn_01x05_Female, J6 Conn_01x05_Male, J7 Conn_01x05_Male, Q1 BC547, Q2 BC547, SW1 SW_Push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

Commit message: Layout and add LED to Kick
Parts:
- added D3: LED, LED_THT:LED_D5.0mm, F.Cu at (52.7, 37.5)
- added R15: 1k, Resistor_THT:R_Axial_DIN0207_L6.3mm_D2.5mm_P10.16mm_Horizontal, B.Cu at (59.7, 59.1)
- moved D1 20.8 mm to (80.0, 54.6)
- moved D2 20.8 mm to (72.4, 62.2)
- moved R3 17.3 mm to (72.4, 37.5)
- moved R7 16.9 mm to (68.6, 34.9)
- moved C2 15.2 mm to (83.8, 61.0)
- moved C4 15.2 mm to (68.6, 60.7)
- moved Q2 15.2 mm to (82.5, 41.3), turned to 90 degrees
- moved R1 15.0 mm to (76.2, 37.5)
- moved R9 14.6 mm to (83.8, 24.8)
- moved C3 13.1 mm to (80.6, 70.5), turned to 270 degrees
- moved R5 12.9 mm to (72.4, 34.9), turned to 90 degrees
- moved R2 7.62 mm to (80.0, 24.8)
- moved C5 4.95 mm to (84.5, 75.6), turned to 90 degrees
- moved R6 3.82 mm to (68.6, 47.6)
- moved U1 3.81 mm to (76.8, 69.6)
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Connections:
- C2 pad 2: Net-(C2-Pad2) -> /LED_PCB_A
- J4 pad 5: Net-(J4-Pad5) -> /LED_PCB_A
- J6 pad 5: Net-(J6-Pad5) -> /LED_PCB_B
- Q2 pad 1: Net-(C2-Pad2) -> /LED_PCB_A
- R5 pad 1: Net-(C2-Pad2) -> /LED_PCB_A
Routing:
- net /GND_PCB_B: track 54.1 -> 0.00 mm
- net /LED_PCB_A: track 0.00 -> 46.5 mm
- net Net-(C2-Pad2): track 36.7 -> 0.00 mm
- net Net-(Q1-Pad1): track 43.8 -> 20.4 mm
- net Net-(C5-Pad1): track 64.1 -> 41.1 mm
- net Net-(D3-Pad1): track 0.00 -> 22.9 mm
- net Net-(R1-Pad1): track 0.00 -> 21.8 mm
- net /LED_PCB_B: track 0.00 -> 19.7 mm
- net Net-(D2-Pad1): track 42.6 -> 54.5 mm
- net /FREQ_PCB_A: track 17.9 -> 6.50 mm
- net +12V: track 100.8 -> 111.9 mm
- net Net-(C3-Pad2): track 30.5 -> 21.7 mm
- net Net-(Q1-Pad3): track 17.1 -> 25.0 mm
- net /FREQ_PCB_B: track 34.2 -> 41.2 mm
- net Net-(C3-Pad1): track 33.8 -> 40.4 mm
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
Commit message: Fix resistor location
Connections:
- R14 pad 2: Net-(C6-Pad1) -> /OUT_PCB_A
Routing:
- net /OUT_PCB_A: track 31.5 -> 39.1 mm
- net Net-(C6-Pad1): track 11.1 -> 8.30 mm
- net -12V: track 71.1 -> 72.2 mm
Changed lines of the file:
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@@
     (thickness 1.6)
     (drawings 8)
-    (tracks 208)
+    (tracks 209)
     (zones 0)
     (modules 41)
@@
     (fp_line (start 1.93 1.25) (end 1.93 -1.25) (layer B.Fab) (width 0.1))
     (pad 2 thru_hole oval (at 10.16 0 270) (size 1.6 1.6) (drill 0.8) (layers *.Cu *.Mask)
-      (net 8 "Net-(C6-Pad1)"))
+      (net 32 /OUT_PCB_A))
     (pad 1 thru_hole circle (at 0 0 270) (size 1.6 1.6) (drill 0.8) (layers *.Cu *.Mask)
       (net 2 GND))
@@
   (segment (start 80.01 54.61) (end 80.01 50.30363) (width 0.25) (layer F.Cu) (net 1))
   (segment (start 77.33137 47.625) (end 76.2 47.625) (width 0.25) (layer F.Cu) (net 1))
-  (segment (start 81.675002 41.275) (end 82.55 41.275) (width 0.25) (layer F.Cu) (net 41))
-  (segment (start 76.740001 36.339999) (end 81.675002 41.275) (width 0.25) (layer F.Cu) (net 41))
-  (segment (start 72.39 34.925) (end 73.804999 36.339999) (width 0.25) (layer F.Cu) (net 41))
-  (segment (start 73.804999 36.339999) (end 76.740001 36.339999) (width 0.25) (layer F.Cu) (net 41))
-  (segment (start 82.55 42.05) (end 82.55 41.275) (width 0.25) (layer B.Cu) (net 41))
-  (segment (start 83.82 55.96) (end 81.024988 53.164988) (width 0.25) (layer B.Cu) (net 41))
-  (segment (start 81.024988 43.575012) (end 82.55 42.05) (width 0.25) (layer B.Cu) (net 41))
-  (segment (start 81.024988 53.164988) (end 81.024988 43.575012) (width 0.25) (layer B.Cu) (net 41))
   (segment (start 69.379999 38.264999) (end 68.58 37.465) (width 0.25) (layer F.Cu) (net 3))
   (segment (start 69.85 38.735) (end 69.379999 38.264999) (width 0.25) (layer F.Cu) (net 3))
@@
   (segment (start 83.329999 74.439999) (end 82.078999 74.439999) (width 0.25) (layer F.Cu) (net 7))
   (segment (start 84.455 75.565) (end 83.329999 74.439999) (width 0.25) (layer F.Cu) (net 7))
-  (segment (start 80.01 93.98) (end 83.82 93.98) (width 0.25) (layer F.Cu) (net 8))
-  (segment (start 80.645 94.615) (end 80.01 93.98) (width 0.25) (layer F.Cu) (net 8))
-  (segment (start 80.645 100.965) (end 80.645 94.615) (width 0.25) (layer F.Cu) (net 8))
+  (segment (start 83.82 97.79) (end 80.645 100.965) (width 0.25) (layer B.Cu) (net 8))
+  (segment (start 83.82 93.98) (end 83.82 97.79) (width 0.25) (layer B.Cu) (net 8))
   (segment (start 74.881314 119.38) (end 73.66 119.38) (width 0.25) (layer F.Cu) (net 9))
   (segment (start 81.560002 119.38) (end 74.881314 119.38) (width 0.25) (layer F.Cu) (net 9))
@@
   (segment (start 72.438686 119.38) (end 71.12 119.38) (width 0.25) (layer F.Cu) (net 9))
   (segment (start 73.66 119.38) (end 72.438686 119.38) (width 0.25) (layer F.Cu) (net 9))
-  (segment (start 76.835 78.266) (end 76.835 77.216) (width 0.25) (layer B.Cu) (net 9))
-  (segment (start 78.285 79.716) (end 76.835 78.266) (width 0.25) (layer B.Cu) (net 9))
-  (segment (start 78.285 90.110002) (end 78.285 79.716) (width 0.25) (layer B.Cu) (net 9))
-  (segment (start 83.770001 95.595003) (end 78.285 90.110002) (width 0.25) (layer B.Cu) (net 9))
-  (segment (start 83.770001 116.984999) (end 83.770001 95.595003) (width 0.25) (layer B.Cu) (net 9))
-  (segment (start 82.645 118.11) (end 83.770001 116.984999) (width 0.25) (layer B.Cu) (net 9))
   (segment (start 74.765001 66.839999) (end 75.565 66.04) (width 0.25) (layer F.Cu) (net 9))
   (segment (start 74.765001 72.057005) (end 74.765001 66.839999) (width 0.25) (layer F.Cu) (net 9))
@@
   (segment (start 77.235 77.216) (end 78.36001 76.09099) (width 0.25) (layer F.Cu) (net 9))
   (segment (start 76.835 77.216) (end 77.235 77.216) (width 0.25) (layer F.Cu) (net 9))
+  (segment (start 76.835 78.266) (end 76.835 77.216) (width 0.25) (layer B.Cu) (net 9))
+  (segment (start 76.835 78.500002) (end 76.835 78.266) (width 0.25) (layer B.Cu) (net 9))
+  (segment (start 85.09 86.755002) (end 76.835 78.500002) (width 0.25) (layer B.Cu) (net 9))
+  (segment (start 85.09 115.665) (end 85.09 86.755002) (width 0.25) (layer B.Cu) (net 9))
+  (segment (start 82.645 118.11) (end 85.09 115.665) (width 0.25) (layer B.Cu) (net 9))
   (segment (start 71.590001 25.564999) (end 72.39 24.765) (width 0.25) (layer F.Cu) (net 10))
   (segment (start 71.12 26.035) (end 71.590001 25.564999) (width 0.25) (layer F.Cu) (net 10))
@@
   (segment (start 82.645 102.09637) (end 83.770001 103.221371) (width 0.25) (layer F.Cu) (net 32))
   (segment (start 82.645 100.965) (end 82.645 102.09637) (width 0.25) (layer F.Cu) (net 32))
+  (segment (start 80.01 97.19863) (end 80.01 94.43001) (width 0.25) (layer F.Cu) (net 32))
+  (segment (start 82.645 100.965) (end 82.645 99.83363) (width 0.25) (layer F.Cu) (net 32))
+  (segment (start 82.645 99.83363) (end 80.01 97.19863) (width 0.25) (layer F.Cu) (net 32))
   (segment (start 53.848 23.017) (end 59.152 28.321) (width 0.25) (layer F.Cu) (net 33))
   (segment (start 53.848 21.336) (end 53.848 23.017) (width 0.25) (layer F.Cu) (net 33))
@@
   (segment (start 49.53 50.736602) (end 52.705 47.561602) (width 0.25) (layer F.Cu) (net 40))
   (segment (start 49.53 59.055) (end 49.53 50.736602) (width 0.25) (layer F.Cu) (net 40))
+  (segment (start 81.675002 41.275) (end 82.55 41.275) (width 0.25) (layer F.Cu) (net 41))
+  (segment (start 76.740001 36.339999) (end 81.675002 41.275) (width 0.25) (layer F.Cu) (net 41))
+  (segment (start 72.39 34.925) (end 73.804999 36.339999) (width 0.25) (layer F.Cu) (net 41))
+  (segment (start 73.804999 36.339999) (end 76.740001 36.339999) (width 0.25) (layer F.Cu) (net 41))
+  (segment (start 82.55 42.05) (end 82.55 41.275) (width 0.25) (layer B.Cu) (net 41))
+  (segment (start 83.82 55.96) (end 81.024988 53.164988) (width 0.25) (layer B.Cu) (net 41))
+  (segment (start 81.024988 43.575012) (end 82.55 42.05) (width 0.25) (layer B.Cu) (net 41))
+  (segment (start 81.024988 53.164988) (end 81.024988 43.575012) (width 0.25) (layer B.Cu) (net 41))
   (segment (start 81.28 26.035) (end 72.39 34.925) (width 0.25) (layer B.Cu) (net 41))
   (segment (start 81.28 21.336) (end 81.28 26.035) (width 0.25) (layer B.Cu) (net 41))

Commit message: Fix reversed capacitor
Parts:
- moved C10 1.91 mm to (82.5, 109.2), turned to 180 degrees
Connections:
- C10 pad 1: GND -> +12V
- C10 pad 2: +12V -> GND
Changed lines of the file:
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@@
   )
   (module Capacitor_THT:CP_Radial_D5.0mm_P2.00mm (layer B.Cu)
-    (at 80.645 109.22)
+    (at 82.55 109.22 180)
     (descr "CP, Radial series, Radial, pin pitch=2.00mm, , diameter=5mm, Electrolytic Capacitor")
     (tags "CP Radial series Radial pin pitch 2.00mm  diameter 5mm Electrolytic Capacitor")
@@
     (fp_circle (center 1 0) (end 3.62 0) (layer B.SilkS) (width 0.12))
     (fp_circle (center 1 0) (end 3.5 0) (layer B.Fab) (width 0.1))
-    (pad 2 thru_hole circle (at 2 0) (size 1.6 1.6) (drill 0.8) (layers *.Cu *.Mask)
+    (pad 2 thru_hole circle (at 2 0 180) (size 1.6 1.6) (drill 0.8) (layers *.Cu *.Mask)
+      (net 2 GND))
+    (pad 1 thru_hole rect (at 0 0 180) (size 1.6 1.6) (drill 0.8) (layers *.Cu *.Mask)
       (net 10 +12V))
-    (pad 1 thru_hole rect (at 0 0) (size 1.6 1.6) (drill 0.8) (layers *.Cu *.Mask)
-      (net 2 GND))
     (model ${KISYS3DMOD}/Capacitor_THT.3dshapes/CP_Radial_D5.0mm_P2.00mm.wrl
       (at (xyz 0 0 0))
