File: wip/mod_synth_lfo_full/schematic/mod_synth_lfo_full.kicad_pcb (KiCad board)
At the start: 2 copper layers, 62.2 x 109.2 mm, 75 parts, among them J1 CV, J2 Conn_02x08_Odd_Even, J3 SIN, J4 COS, J5 TRI, J6 SQR, J7 RAMP UP, J8 RAMP DOWN, Q1 BC550, Q2 BC550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

Commit message: Reverse pots
Connections:
- RV1 pad 1: +12V -> GND
- RV1 pad 3: GND -> +12V
- RV2 pad 1: Net-(J1-PadT) -> GND
- RV2 pad 3: GND -> Net-(J1-PadT)
Changed lines of the file:
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@@
     (pad "" thru_hole circle (at 7.5 7.3 180) (size 3.24 3.24) (drill 1.8) (layers *.Cu *.Mask))
     (pad 3 thru_hole circle (at 0 5 180) (size 1.8 1.8) (drill 1) (layers *.Cu *.Mask)
-      (net 1 GND))
+      (net 7 "Net-(J1-PadT)"))
     (pad 2 thru_hole circle (at 0 2.5 180) (size 1.8 1.8) (drill 1) (layers *.Cu *.Mask)
       (net 34 "Net-(R2-Pad2)"))
     (pad 1 thru_hole rect (at 0 0 180) (size 1.8 1.8) (drill 1) (layers *.Cu *.Mask)
-      (net 7 "Net-(J1-PadT)"))
+      (net 1 GND))
     (model ${KISYS3DMOD}/Potentiometer_THT.3dshapes/Potentiometer_Alpha_RD901F-40-00D_Single_Vertical.wrl
       (at (xyz 0 0 0))
@@
     (pad "" thru_hole circle (at 7.5 7.3 180) (size 3.24 3.24) (drill 1.8) (layers *.Cu *.Mask))
     (pad 3 thru_hole circle (at 0 5 180) (size 1.8 1.8) (drill 1) (layers *.Cu *.Mask)
-      (net 1 GND))
+      (net 2 +12V))
     (pad 2 thru_hole circle (at 0 2.5 180) (size 1.8 1.8) (drill 1) (layers *.Cu *.Mask)
       (net 32 "Net-(R1-Pad2)"))
     (pad 1 thru_hole rect (at 0 0 180) (size 1.8 1.8) (drill 1) (layers *.Cu *.Mask)
-      (net 2 +12V))
+      (net 1 GND))
     (model ${KISYS3DMOD}/Potentiometer_THT.3dshapes/Potentiometer_Alpha_RD901F-40-00D_Single_Vertical.wrl
       (at (xyz 0 0 0))
