File: wip/mod_synth_lfo_full/schematic/mod_synth_lfo_full.sch (KiCad schematic (older format))
At the start: 75 parts, among them J1 CV, J2 Conn_02x08_Odd_Even, J3 SIN, J4 COS, J5 TRI, J6 SQR, J7 RAMP UP, J8 RAMP DOWN, Q1 BC550, Q2 BC550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

Commit message: Reverse pots
Connections:
- net +12V: now also RV1.3; no longer RV1.1
- net GND: now also RV1.1, RV2.1; no longer RV1.3, RV2.3
- net at J1.T: now also RV2.3; no longer RV2.1
Changed lines of the file:
@@
 F 3 "~" H 1100 3450 50  0001 C CNN
 	1    1100 3450
-	1    0    0    -1
+	1    0    0    1
 $EndComp
 $Comp
@@
 F 3 "~" H 1325 4025 50  0001 C CNN
 	1    1325 4025
-	0    -1   -1   0
+	0    1    -1   0
 $EndComp
 $Comp
