File: mod_synth_adsr/schematic/mod_synth_adsr.sch (KiCad schematic (older format))
At the start: 31 parts

Commit message: Add footprints
Parts:
- added C4, C5: CP_Small, Capacitor_THT:CP_Radial_D5.0mm_P2.00mm, symbol Device:CP_Small
- added C6, C7, C8, C9: C_Small, Capacitor_THT:C_Disc_D9.0mm_W2.5mm_P5.00mm, symbol Device:C_Small
- added J3: Conn_02x08_Odd_Even, Connector_IDC:IDC-Header_2x08_P2.54mm_Vertical, symbol Connector_Generic:Conn_02x08_Odd_Even
- C1, C2, C3: renamed from C?; footprint (none) -> Capacitor_THT:C_Disc_D9.0mm_W2.5mm_P5.00mm
- J1, J2: renamed from J?; footprint (none) -> Connector_Audio:Jack_3.5mm_QingPu_WQP-PJ398SM_Vertical_CircularHoles
- R1, R10, R2, R3, R4, R5, R6, R7, R8, R9: renamed from R?; footprint (none) -> Resistor_THT:R_Axial_DIN0207_L6.3mm_D2.5mm_P10.16mm_Horizontal
- RV1, RV2, RV3, RV4: renamed from RV?; footprint (none) -> Potentiometer_THT:Potentiometer_Alpha_RD901F-40-00D_Single_Vertical_CircularHoles
- U1, U2: renamed from U?; footprint (none) -> Package_DIP:DIP-8_W7.62mm_Socket_LongPads
- gave numbers to parts that had none: 9
Connections:
- net +12V: now also U1.8 (V+), C5.1, C7.2, C9.2, J3.10 (Pin_10), J3.9 (Pin_9)
- net GND: now also C4.1, C5.2, C6.2, C7.1, C8.2, C9.1, J3.3 (Pin_3), J3.4 (Pin_4), J3.5 (Pin_5), J3.6 (Pin_6), J3.7 (Pin_7), J3.8 (Pin_8)
- net at U1.6 (-): now also J2.T, U1.7
- net -12V: now reaches U1.4 (V-)
- net -12V: now also C4.2, C6.1, C8.1, J3.1 (Pin_1), J3.2 (Pin_2)
Other:
- moved on the sheet: U1C
